File: box/Schematics/v3/dsp.sch (KiCad schematic (older format))
At the start: 9 parts, among them U2 FOX924B, U5 STM32F373CCT6

Commit message: Moved brokers to rust with mongo reporting
Parts:
- C14, C15, C16, C17, C18, C19, C20: symbol C -> opqbox3-rescue:C
- U2: symbol FOX924B -> opqbox3-rescue:FOX924B
- U5: symbol STM32F373CCT6 -> opqbox3-rescue:STM32F373CCT6
Changed lines of the file:
@@
-EESchema Schematic File Version 2
-LIBS:opqbox3
-LIBS:device
-LIBS:power
-LIBS:conn
+EESchema Schematic File Version 4
 LIBS:opqbox3-cache
-EELAYER 25 0
+EELAYER 26 0
 EELAYER END
 $Descr A4 11693 8268
@@
 $EndDescr
 $Comp
-L GND #PWR024
+L power:GND #PWR024
 U 1 1 5A82B565
 P 2500 3850
@@
 $EndComp
 $Comp
-L +3.3V #PWR025
+L power:+3.3V #PWR025
 U 1 1 5A82B58A
 P 2500 3350
@@
 $EndComp
 $Comp
-L C C14
+L opqbox3-rescue:C C14
 U 1 1 5A82B5B1
 P 2250 3600
@@
 PPS
 $Comp
-L GND #PWR026
+L power:GND #PWR026
 U 1 1 5A82E118
 P 5050 6000
@@
 LED1
 $Comp
-L C C20
+L opqbox3-rescue:C C20
 U 1 1 5A82E38B
 P 6400 1650
@@
 $EndComp
 $Comp
-L GND #PWR027
+L power:GND #PWR027
 U 1 1 5A82E58F
 P 6400 1800
@@
 BOOT_MODE
 $Comp
-L C C15
+L opqbox3-rescue:C C15
 U 1 1 5A82EBD3
 P 4350 1250
@@
 $EndComp
 $Comp
-L C C16
+L opqbox3-rescue:C C16
 U 1 1 5A82EC66
 P 4600 1250
@@
 $EndComp
 $Comp
-L GND #PWR028
+L power:GND #PWR028
 U 1 1 5A82EC8F
 P 4350 1500
@@
 $EndComp
 $Comp
-L +3.3V #PWR029
+L power:+3.3V #PWR029
 U 1 1 5A82EF25
 P 4350 950
@@
 $EndComp
 $Comp
-L C C17
+L opqbox3-rescue:C C17
 U 1 1 5A82F121
 P 5100 1250
@@
 $EndComp
 $Comp
-L C C18
+L opqbox3-rescue:C C18
 U 1 1 5A82F587
 P 5700 1200
@@
 $EndComp
 $Comp
-L C C19
+L opqbox3-rescue:C C19
 U 1 1 5A82F58D
 P 5950 1200
@@
 $EndComp
 $Comp
-L +3.3V #PWR030
+L power:+3.3V #PWR030
 U 1 1 5A82FBC9
 P 5100 950
@@
 $EndComp
 $Comp
-L +3.3V #PWR031
+L power:+3.3V #PWR031
 U 1 1 5A82FBEF
 P 5950 950
@@
 JTAG_JTMS
 $Comp
-L FOX924B U2
+L opqbox3-rescue:FOX924B U2
 U 1 1 5A83A700
 P 2600 3550
@@
 	5050 1750 5050 1850
 $Comp
-L +3.3V #PWR032
+L power:+3.3V #PWR032
 U 1 1 5A8304E4
 P 5050 1750
@@
 $EndComp
 $Comp
-L STM32F373CCT6 U5
+L opqbox3-rescue:STM32F373CCT6 U5
 U 1 1 5A835F5B
 P 3750 3350
