File: box/Schematics/v3/io.sch (KiCad schematic (older format))
At the start: 9 parts, among them J3 Conn_02x20_Odd_Even, J4 Conn_02x04_Odd_Even, J5 Conn_01x04

Commit message: start layout
Parts:
- D1, D2, D3: footprint (none) -> LEDs:LED_0603_HandSoldering
- J3: footprint (none) -> Pin_Headers:Pin_Header_Straight_2x20_Pitch2.54mm
- J4: footprint (none) -> Pin_Headers:Pin_Header_Straight_2x04_Pitch1.00mm
- J5: footprint (none) -> Pin_Headers:Pin_Header_Straight_1x04_Pitch2.54mm
- R11, R12, R13: value R -> 68; footprint (none) -> Resistors_SMD:R_0402
Changed lines of the file:
@@
 EESchema Schematic File Version 2
+LIBS:opqbox3-rescue
 LIBS:opqbox3
 LIBS:device
@@
 F 0 "J3" H 2250 3350 50  0000 C CNN
 F 1 "Conn_02x20_Odd_Even" H 2250 1250 50  0000 C CNN
-F 2 "" H 2200 2350 50  0001 C CNN
+F 2 "Pin_Headers:Pin_Header_Straight_2x20_Pitch2.54mm" H 2200 2350 50  0001 C CNN
 F 3 "" H 2200 2350 50  0001 C CNN
 	1    2200 2350
@@
 F 0 "J4" H 4350 1750 50  0000 C CNN
 F 1 "Conn_02x04_Odd_Even" H 4350 1250 50  0000 C CNN
-F 2 "" H 4300 1550 50  0001 C CNN
+F 2 "Pin_Headers:Pin_Header_Straight_2x04_Pitch1.00mm" H 4300 1550 50  0001 C CNN
 F 3 "" H 4300 1550 50  0001 C CNN
 	1    4300 1550
@@
 F 0 "J5" H 4700 2950 50  0000 C CNN
 F 1 "Conn_01x04" H 4700 2450 50  0000 C CNN
-F 2 "" H 4700 2750 50  0001 C CNN
+F 2 "Pin_Headers:Pin_Header_Straight_1x04_Pitch2.54mm" H 4700 2750 50  0001 C CNN
 F 3 "" H 4700 2750 50  0001 C CNN
 	1    4700 2750
@@
 F 0 "D1" H 6600 1600 50  0000 C CNN
 F 1 "LED" H 6600 1400 50  0000 C CNN
-F 2 "" H 6600 1500 50  0001 C CNN
+F 2 "LEDs:LED_0603_HandSoldering" H 6600 1500 50  0001 C CNN
 F 3 "" H 6600 1500 50  0001 C CNN
 	1    6600 1500
@@
 F 0 "D2" H 6600 1900 50  0000 C CNN
 F 1 "LED" H 6600 1700 50  0000 C CNN
-F 2 "" H 6600 1800 50  0001 C CNN
+F 2 "LEDs:LED_0603_HandSoldering" H 6600 1800 50  0001 C CNN
 F 3 "" H 6600 1800 50  0001 C CNN
 	1    6600 1800
@@
 F 0 "D3" H 6600 2200 50  0000 C CNN
 F 1 "LED" H 6600 2000 50  0000 C CNN
-F 2 "" H 6600 2100 50  0001 C CNN
+F 2 "LEDs:LED_0603_HandSoldering" H 6600 2100 50  0001 C CNN
 F 3 "" H 6600 2100 50  0001 C CNN
 	1    6600 2100
@@
 P 6250 1500
 F 0 "R11" V 6330 1500 50  0000 C CNN
-F 1 "R" V 6250 1500 50  0000 C CNN
-F 2 "" V 6180 1500 50  0001 C CNN
+F 1 "68" V 6250 1500 50  0000 C CNN
+F 2 "Resistors_SMD:R_0402" V 6180 1500 50  0001 C CNN
 F 3 "" H 6250 1500 50  0001 C CNN
 	1    6250 1500
@@
 P 6250 1800
 F 0 "R12" V 6330 1800 50  0000 C CNN
-F 1 "R" V 6250 1800 50  0000 C CNN
-F 2 "" V 6180 1800 50  0001 C CNN
+F 1 "68" V 6250 1800 50  0000 C CNN
+F 2 "Resistors_SMD:R_0402" V 6180 1800 50  0001 C CNN
 F 3 "" H 6250 1800 50  0001 C CNN
 	1    6250 1800
@@
 P 6250 2100
 F 0 "R13" V 6330 2100 50  0000 C CNN
-F 1 "R" V 6250 2100 50  0000 C CNN
-F 2 "" V 6180 2100 50  0001 C CNN
+F 1 "68" V 6250 2100 50  0000 C CNN
+F 2 "Resistors_SMD:R_0402" V 6180 2100 50  0001 C CNN
 F 3 "" H 6250 2100 50  0001 C CNN
 	1    6250 2100

Commit message: add chip pro and battery
Parts:
- removed J3: Conn_02x20_Odd_Even, Pin_Headers:Pin_Header_Straight_2x20_Pitch2.54mm, symbol Conn_02x20_Odd_Even
Connections:
- net labels removed: BOOT_MODE, FLAG1, SPI_CLK, SPI_MISO, SPI_MOSI, SPI_nCS, UART_RX, UART_TX
- wire segments 29 -> 20
- no-connect marks 27 -> 1
Other:
- note removed: "RPi Header"
- moved on the sheet: D1, D2, D3, J4, J5, R11, R12, R13

Commit message: remove chip, replace pi
Parts:
- J4: footprint Pin_Headers:Pin_Header_Straight_2x04_Pitch1.00mm -> Pin_Headers:Pin_Header_Straight_2x04_Pitch2.54mm
Changed lines of the file:
@@
 F 0 "J4" H 1600 1400 50  0000 C CNN
 F 1 "Conn_02x04_Odd_Even" H 1600 900 50  0000 C CNN
-F 2 "Pin_Headers:Pin_Header_Straight_2x04_Pitch1.00mm" H 1550 1200 50  0001 C CNN
+F 2 "Pin_Headers:Pin_Header_Straight_2x04_Pitch2.54mm" H 1550 1200 50  0001 C CNN
 F 3 "" H 1550 1200 50  0001 C CNN
 	1    1550 1200
@@
 NoConn ~ 1350 1100
 $Comp
-L GND #PWR044
+L GND #PWR035
 U 1 1 5A852BF5
 P 2050 950
-F 0 "#PWR044" H 2050 700 50  0001 C CNN
+F 0 "#PWR035" H 2050 700 50  0001 C CNN
 F 1 "GND" H 2050 800 50  0000 C CNN
 F 2 "" H 2050 950 50  0001 C CNN
@@
 $EndComp
 $Comp
-L GND #PWR045
+L GND #PWR036
 U 1 1 5A857B5F
 P 1650 2700
-F 0 "#PWR045" H 1650 2450 50  0001 C CNN
+F 0 "#PWR036" H 1650 2450 50  0001 C CNN
 F 1 "GND" H 1650 2550 50  0000 C CNN
 F 2 "" H 1650 2700 50  0001 C CNN
@@
 Connection ~ 1650 2600
 $Comp
-L +5V #PWR046
+L +5V #PWR037
 U 1 1 5A857BAF
 P 1650 2250
-F 0 "#PWR046" H 1650 2100 50  0001 C CNN
+F 0 "#PWR037" H 1650 2100 50  0001 C CNN
 F 1 "+5V" H 1650 2390 50  0000 C CNN
 F 2 "" H 1650 2250 50  0001 C CNN
@@
 $EndComp
 $Comp
-L GND #PWR047
+L GND #PWR038
 U 1 1 5A85F4E9
 P 4100 1850
-F 0 "#PWR047" H 4100 1600 50  0001 C CNN
+F 0 "#PWR038" H 4100 1600 50  0001 C CNN
 F 1 "GND" H 4100 1700 50  0000 C CNN
 F 2 "" H 4100 1850 50  0001 C CNN
@@
 	3300 1450 3350 1450
 $Comp
-L +5V #PWR048
+L +5V #PWR039
 U 1 1 5A85F8C1
 P 3250 1100
-F 0 "#PWR048" H 3250 950 50  0001 C CNN
+F 0 "#PWR039" H 3250 950 50  0001 C CNN
 F 1 "+5V" H 3250 1240 50  0000 C CNN
 F 2 "" H 3250 1100 50  0001 C CNN

Commit message: Moved brokers to rust with mongo reporting
Parts:
- D1, D2, D3: symbol LED -> opqbox3-rescue:LED
- J4: symbol Conn_02x04_Odd_Even -> opqbox3-rescue:Conn_02x04_Odd_Even
- J5: symbol Conn_01x04 -> opqbox3-rescue:Conn_01x04
- R11, R12, R13: symbol R -> opqbox3-rescue:R
Changed lines of the file:
@@
-EESchema Schematic File Version 2
-LIBS:opqbox3
-LIBS:device
-LIBS:power
-LIBS:conn
+EESchema Schematic File Version 4
 LIBS:opqbox3-cache
-EELAYER 25 0
+EELAYER 26 0
 EELAYER END
 $Descr A4 11693 8268
@@
 JTAG Header
 $Comp
-L Conn_02x04_Odd_Even J4
+L opqbox3-rescue:Conn_02x04_Odd_Even J4
 U 1 1 5A852B85
 P 1550 1200
@@
 NoConn ~ 1350 1100
 $Comp
-L GND #PWR035
+L power:GND #PWR035
 U 1 1 5A852BF5
 P 2050 950
@@
 	2050 900  2050 950
 $Comp
-L Conn_01x04 J5
+L opqbox3-rescue:Conn_01x04 J5
 U 1 1 5A857B11
 P 1950 2400
@@
 $EndComp
 $Comp
-L GND #PWR036
+L power:GND #PWR036
 U 1 1 5A857B5F
 P 1650 2700
@@
 $EndComp
 Wire Wire Line
-	1650 2500 1650 2700
+	1650 2500 1650 2600
 Wire Wire Line
 	1750 2600 1650 2600
@@
 Connection ~ 1650 2600
 $Comp
-L +5V #PWR037
+L power:+5V #PWR037
 U 1 1 5A857BAF
 P 1650 2250
@@
 4 Pos Header
 $Comp
-L LED D1
+L opqbox3-rescue:LED D1
 U 1 1 5A85F2BE
 P 3850 1150
@@
 $EndComp
 $Comp
-L LED D2
+L opqbox3-rescue:LED D2
 U 1 1 5A85F345
 P 3850 1450
@@
 $EndComp
 $Comp
-L LED D3
+L opqbox3-rescue:LED D3
 U 1 1 5A85F3E5
 P 3850 1750
@@
 $EndComp
 $Comp
-L R R11
+L opqbox3-rescue:R R11
 U 1 1 5A85F458
 P 3500 1150
@@
 $EndComp
 $Comp
-L R R12
+L opqbox3-rescue:R R12
 U 1 1 5A85F48B
 P 3500 1450
@@
 $EndComp
 $Comp
-L R R13
+L opqbox3-rescue:R R13
 U 1 1 5A85F4B8
 P 3500 1750
@@
 $EndComp
 $Comp
-L GND #PWR038
+L power:GND #PWR038
 U 1 1 5A85F4E9
 P 4100 1850
@@
 $EndComp
 Wire Wire Line
-	4100 1150 4100 1850
+	4100 1150 4100 1450
 Wire Wire Line
 	4100 1750 4000 1750
@@
 	3300 1450 3350 1450
 $Comp
-L +5V #PWR039
+L power:+5V #PWR039
 U 1 1 5A85F8C1
 P 3250 1100
@@
 Wire Wire Line
 	3250 1150 3350 1150
+Wire Wire Line
+	1650 2600 1650 2700
+Wire Wire Line
+	4100 1750 4100 1850
+Wire Wire Line
+	4100 1450 4100 1750
 $EndSCHEMATC
