File: box/Schematics/v3/pi.sch (KiCad schematic (older format))
At the start: 1 part, among them J3 Raspberry_Pi_2_3

Commit message: add IRM-15-05 and replace 05
Parts:
- J3: footprint Pin_Headers:Pin_Header_Straight_2x20 -> Pin_Headers:Pin_Header_Straight_2x20_Pitch2.54mm
Changed lines of the file:
@@
 UART_RX
 $Comp
-L GND #PWR033
+L GND #PWR29
 U 1 1 5A9AD0C2
 P 6050 5400
-F 0 "#PWR033" H 6050 5150 50  0001 C CNN
+F 0 "#PWR29" H 6050 5150 50  0001 C CNN
 F 1 "GND" H 6050 5250 50  0000 C CNN
 F 2 "" H 6050 5400 50  0001 C CNN
@@
 JTAG_nRST
 $Comp
-L +5V #PWR034
+L +5V #PWR28
 U 1 1 5A9B4CD7
 P 5950 2600
-F 0 "#PWR034" H 5950 2450 50  0001 C CNN
+F 0 "#PWR28" H 5950 2450 50  0001 C CNN
 F 1 "+5V" H 5950 2740 50  0000 C CNN
 F 2 "" H 5950 2600 50  0001 C CNN
@@
 F 0 "J3" H 6800 2750 50  0000 C CNN
 F 1 "Raspberry_Pi_2_3" H 5700 4900 50  0000 C CNN
-F 2 "Pin_Headers:Pin_Header_Straight_2x20" H 7100 5250 50  0001 C CNN
+F 2 "Pin_Headers:Pin_Header_Straight_2x20_Pitch2.54mm" H 7100 5250 50  0001 C CNN
 F 3 "" H 6150 3850 50  0001 C CNN
 	1    6100 4000

Commit message: Moved brokers to rust with mongo reporting
Parts:
- added J?: Conn_01x04, Pin_Headers:Pin_Header_Straight_1x04_Pitch2.54mm, symbol opqbox3-rescue:Conn_01x04
- added R10, R11: 665, Resistors_SMD:R_0402, symbol opqbox3-rescue:R
- J3: symbol Raspberry_Pi_2_3 -> opqbox3-rescue:Raspberry_Pi_2_3
Connections:
- net GND: now also J?.4 (Pin_4)
- net SPI_MISO: now also J3.19 ((SPI_MOSI)_GPIO10); no longer J3.21 ((SPI_MISO)_GPIO9)
- net SPI_MOSI: now also J3.21 ((SPI_MISO)_GPIO9); no longer J3.19 ((SPI_MOSI)_GPIO10)
- net at J3.1 (3V3): now also J?.1 (Pin_1), R10.2, R11.2
- net at J3.3 ((SDA1)_GPIO2): now also J?.2 (Pin_2), R10.1
- net at J3.5 ((SCL1)_GPIO3): now also J?.3 (Pin_3), R11.1
Changed lines of the file:
@@
-EESchema Schematic File Version 2
-LIBS:opqbox3
-LIBS:device
-LIBS:power
-LIBS:conn
+EESchema Schematic File Version 4
 LIBS:opqbox3-cache
-EELAYER 25 0
+EELAYER 26 0
 EELAYER END
 $Descr A4 11693 8268
@@
 Comment4 ""
 $EndDescr
-Text HLabel 7000 4100 2    60   Output ~ 0
+Text HLabel 7000 4000 2    60   Output ~ 0
 SPI_MOSI
-Text HLabel 7000 4000 2    60   Input ~ 0
+Text HLabel 7000 4100 2    60   Input ~ 0
 SPI_MISO
 Text HLabel 7000 3900 2    60   Output ~ 0
@@
 UART_RX
 $Comp
-L GND #PWR033
+L power:GND #PWR033
 U 1 1 5A9AD0C2
 P 6050 5400
@@
 JTAG_nRST
 $Comp
-L +5V #PWR034
+L power:+5V #PWR034
 U 1 1 5A9B4CD7
 P 5950 2600
@@
 $EndComp
 $Comp
-L Raspberry_Pi_2_3 J3
+L opqbox3-rescue:Raspberry_Pi_2_3 J3
 U 1 1 5AC2C93D
 P 6100 4000
@@
 	5900 2700 5900 2650
 Wire Wire Line
-	5900 2650 6000 2650
+	5900 2650 5950 2650
 Wire Wire Line
 	5950 2650 5950 2600
@@
 	5700 5300 5700 5350
 Wire Wire Line
-	5700 5350 6400 5350
+	5700 5350 5800 5350
 Wire Wire Line
 	6050 5350 6050 5400
@@
 NoConn ~ 6200 2700
 NoConn ~ 6300 2700
+Wire Wire Line
+	5950 2650 6000 2650
+Wire Wire Line
+	6050 5350 6100 5350
+Wire Wire Line
+	5800 5350 5900 5350
+Wire Wire Line
+	5900 5350 6000 5350
+Wire Wire Line
+	6000 5350 6050 5350
+Wire Wire Line
+	6100 5350 6200 5350
+Wire Wire Line
+	6200 5350 6300 5350
+Wire Wire Line
+	6300 5350 6400 5350
+$Comp
+L opqbox3-rescue:Conn_01x04 J?
+U 1 1 5CB6D89C
+P 7750 3100
+AR Path="/5A8506F3/5CB6D89C" Ref="J?"  Part="1"
+AR Path="/5A9ABA19/5CB6D89C" Ref="J?"  Part="1"
+F 0 "J?" H 7750 3300 50  0000 C CNN
+F 1 "Conn_01x04" H 8050 3050 50  0000 C CNN
+F 2 "Pin_Headers:Pin_Header_Straight_1x04_Pitch2.54mm" H 7750 3100 50  0001 C CNN
+F 3 "" H 7750 3100 50  0001 C CNN
+	1    7750 3100
+	1    0    0    -1
+$EndComp
+$Comp
+L power:GND #PWR?
+U 1 1 5CB6DA59
+P 7450 3500
+F 0 "#PWR?" H 7450 3250 50  0001 C CNN
+F 1 "GND" H 7450 3350 50  0000 C CNN
+F 2 "" H 7450 3500 50  0001 C CNN
+F 3 "" H 7450 3500 50  0001 C CNN
+	1    7450 3500
+	1    0    0    -1
+$EndComp
+Wire Wire Line
+	7550 3300 7450 3300
+Wire Wire Line
+	7450 3300 7450 3500
+Wire Wire Line
+	7550 3200 7400 3200
+Wire Wire Line
+	7000 3100 7250 3100
+Wire Wire Line
+	6200 2700 6200 2550
+Wire Wire Line
+	6200 2550 7250 2550
+Wire Wire Line
+	7550 2550 7550 3000
+$Comp
+L opqbox3-rescue:R R?
+U 1 1 5CB74D6F
+P 7250 2950
+AR Path="/5A829EE9/5CB74D6F" Ref="R?"  Part="1"
+AR Path="/5A9ABA19/5CB74D6F" Ref="R10"  Part="1"
+F 0 "R10" V 7330 2950 50  0000 C CNN
+F 1 "665" V 7250 2950 50  0000 C CNN
+F 2 "Resistors_SMD:R_0402" V 7180 2950 50  0001 C CNN
+F 3 "" H 7250 2950 50  0001 C CNN
+	1    7250 2950
+	-1   0    0    1
+$EndComp
+Connection ~ 7250 3100
+Wire Wire Line
+	7250 3100 7550 3100
+$Comp
+L opqbox3-rescue:R R?
+U 1 1 5CB75360
+P 7400 3050
+AR Path="/5A829EE9/5CB75360" Ref="R?"  Part="1"
+AR Path="/5A9ABA19/5CB75360" Ref="R11"  Part="1"
+F 0 "R11" V 7480 3050 50  0000 C CNN
+F 1 "665" V 7400 3050 50  0000 C CNN
+F 2 "Resistors_SMD:R_0402" V 7330 3050 50  0001 C CNN
+F 3 "" H 7400 3050 50  0001 C CNN
+	1    7400 3050
+	-1   0    0    1
+$EndComp
+Connection ~ 7400 3200
+Wire Wire Line
+	7400 3200 7000 3200
+Wire Wire Line
+	7400 2550 7400 2900
+Connection ~ 7400 2550
+Wire Wire Line
+	7400 2550 7550 2550
+Wire Wire Line
+	7250 2800 7250 2550
+Connection ~ 7250 2550
+Wire Wire Line
+	7250 2550 7400 2550
 $EndSCHEMATC
