File: box/Schematics/v3/power.sch (KiCad schematic (older format))
At the start: 31 parts, among them U1 AMC1100DWV, U3 ISL21010CFH333Z-TK

Commit message: update footpring in pcb
Parts:
- PSU1: footprint (none) -> opqbox3:IRM-15-5
Changed lines of the file:
@@
 $EndComp
 $Comp
-L GND #PWR7
+L GND #PWR03
 U 1 1 5A829FB7
 P 4300 1850
-F 0 "#PWR7" H 4300 1600 50  0001 C CNN
+F 0 "#PWR03" H 4300 1600 50  0001 C CNN
 F 1 "GND" H 4300 1700 50  0000 C CNN
 F 2 "" H 4300 1850 50  0001 C CNN
@@
 $EndComp
 $Comp
-L +5V #PWR13
+L +5V #PWR04
 U 1 1 5A829FBB
 P 4900 1300
-F 0 "#PWR13" H 4900 1150 50  0001 C CNN
+F 0 "#PWR04" H 4900 1150 50  0001 C CNN
 F 1 "+5V" H 4900 1440 50  0000 C CNN
 F 2 "" H 4900 1300 50  0001 C CNN
@@
 L_MEASURE
 $Comp
-L NEUT #PWR2
+L NEUT #PWR05
 U 1 1 5A829FBC
 P 2050 2000
-F 0 "#PWR2" H 2050 1850 50  0001 C CNN
+F 0 "#PWR05" H 2050 1850 50  0001 C CNN
 F 1 "NEUT" H 2050 2150 50  0000 C CNN
 F 2 "" H 2050 2000 50  0001 C CNN
@@
 $EndComp
 $Comp
-L LINE #PWR1
+L LINE #PWR06
 U 1 1 5A829FBD
 P 2050 1450
-F 0 "#PWR1" H 2050 1300 50  0001 C CNN
+F 0 "#PWR06" H 2050 1300 50  0001 C CNN
 F 1 "LINE" H 2050 1600 50  0000 C CNN
 F 2 "" H 2050 1450 50  0001 C CNN
@@
 $EndComp
 $Comp
-L PWR_FLAG #FLG3
+L PWR_FLAG #FLG07
 U 1 1 5A829FC1
 P 2900 1350
-F 0 "#FLG3" H 2900 1425 50  0001 C CNN
+F 0 "#FLG07" H 2900 1425 50  0001 C CNN
 F 1 "PWR_FLAG" H 2900 1500 50  0000 C CNN
 F 2 "" H 2900 1350 50  0001 C CNN
@@
 $EndComp
 $Comp
-L PWR_FLAG #FLG5
+L PWR_FLAG #FLG08
 U 1 1 5A829FC2
 P 5200 1300
-F 0 "#FLG5" H 5200 1375 50  0001 C CNN
+F 0 "#FLG08" H 5200 1375 50  0001 C CNN
 F 1 "PWR_FLAG" H 5200 1450 50  0000 C CNN
 F 2 "" H 5200 1300 50  0001 C CNN
@@
 $EndComp
 $Comp
-L NEUT #PWR5
+L NEUT #PWR09
 U 1 1 5A829FC9
 P 2650 4700
-F 0 "#PWR5" H 2650 4550 50  0001 C CNN
+F 0 "#PWR09" H 2650 4550 50  0001 C CNN
 F 1 "NEUT" H 2650 4850 50  0000 C CNN
 F 2 "" H 2650 4700 50  0001 C CNN
@@
 $EndComp
 $Comp
-L NEUT #PWR4
+L NEUT #PWR010
 U 1 1 5A829FCE
 P 2650 3600
-F 0 "#PWR4" H 2650 3450 50  0001 C CNN
+F 0 "#PWR010" H 2650 3450 50  0001 C CNN
 F 1 "NEUT" H 2650 3750 50  0000 C CNN
 F 2 "" H 2650 3600 50  0001 C CNN
@@
 $EndComp
 $Comp
-L NEUT #PWR6
+L NEUT #PWR011
 U 1 1 5A829FD1
 P 3050 5850
-F 0 "#PWR6" H 3050 5700 50  0001 C CNN
+F 0 "#PWR011" H 3050 5700 50  0001 C CNN
 F 1 "NEUT" H 3050 6000 50  0000 C CNN
 F 2 "" H 3050 5850 50  0001 C CNN
@@
 $EndComp
 $Comp
-L NEUT #PWR3
+L NEUT #PWR012
 U 1 1 5A829FD4
 P 2400 6850
-F 0 "#PWR3" H 2400 6700 50  0001 C CNN
+F 0 "#PWR012" H 2400 6700 50  0001 C CNN
 F 1 "NEUT" H 2400 7000 50  0000 C CNN
 F 2 "" H 2400 6850 50  0001 C CNN
@@
 NOT isolated
 $Comp
-L GND #PWR11
+L GND #PWR013
 U 1 1 5A829FD5
 P 4450 6850
-F 0 "#PWR11" H 4450 6600 50  0001 C CNN
+F 0 "#PWR013" H 4450 6600 50  0001 C CNN
 F 1 "GND" H 4450 6700 50  0000 C CNN
 F 2 "" H 4450 6850 50  0001 C CNN
@@
 $EndComp
 $Comp
-L +5V #PWR10
+L +5V #PWR014
 U 1 1 5A829FD7
 P 4450 5700
-F 0 "#PWR10" H 4450 5550 50  0001 C CNN
+F 0 "#PWR014" H 4450 5550 50  0001 C CNN
 F 1 "+5V" H 4450 5840 50  0000 C CNN
 F 2 "" H 4450 5700 50  0001 C CNN
@@
 $EndComp
 $Comp
-L GND #PWR8
+L GND #PWR015
 U 1 1 5A829FDA
 P 4350 4300
-F 0 "#PWR8" H 4350 4050 50  0001 C CNN
+F 0 "#PWR015" H 4350 4050 50  0001 C CNN
 F 1 "GND" H 4350 4150 50  0000 C CNN
 F 2 "" H 4350 4300 50  0001 C CNN
@@
 $EndComp
 $Comp
-L +3.3V #PWR12
+L +3.3V #PWR016
 U 1 1 5A829FDB
 P 4650 3150
-F 0 "#PWR12" H 4650 3000 50  0001 C CNN
+F 0 "#PWR016" H 4650 3000 50  0001 C CNN
 F 1 "+3.3V" H 4650 3290 50  0000 C CNN
 F 2 "" H 4650 3150 50  0001 C CNN
@@
 $EndComp
 $Comp
-L GND #PWR9
+L GND #PWR017
 U 1 1 5A829FE0
 P 4400 3600
-F 0 "#PWR9" H 4400 3350 50  0001 C CNN
+F 0 "#PWR017" H 4400 3350 50  0001 C CNN
 F 1 "GND" H 4400 3450 50  0000 C CNN
 F 2 "" H 4400 3600 50  0001 C CNN
@@
 NEUTRAL
 $Comp
-L PWR_FLAG #FLG4
+L PWR_FLAG #FLG018
 U 1 1 5A83249D
 P 4900 1850
-F 0 "#FLG4" H 4900 1925 50  0001 C CNN
+F 0 "#FLG018" H 4900 1925 50  0001 C CNN
 F 1 "PWR_FLAG" H 4900 2000 50  0000 C CNN
 F 2 "" H 4900 1850 50  0001 C CNN
@@
 $EndComp
 $Comp
-L +5V #PWR14
+L +5V #PWR019
 U 1 1 5A82BC82
 P 6700 1150
-F 0 "#PWR14" H 6700 1000 50  0001 C CNN
+F 0 "#PWR019" H 6700 1000 50  0001 C CNN
 F 1 "+5V" H 6700 1290 50  0000 C CNN
 F 2 "" H 6700 1150 50  0001 C CNN
@@
 Connection ~ 8200 1500
 $Comp
-L GND #PWR16
+L GND #PWR020
 U 1 1 5A82C977
 P 7450 2300
-F 0 "#PWR16" H 7450 2050 50  0001 C CNN
+F 0 "#PWR020" H 7450 2050 50  0001 C CNN
 F 1 "GND" H 7450 2150 50  0000 C CNN
 F 2 "" H 7450 2300 50  0001 C CNN
@@
 $EndComp
 $Comp
-L GND #PWR17
+L GND #PWR021
 U 1 1 5AC2E311
 P 7550 4550
-F 0 "#PWR17" H 7550 4300 50  0001 C CNN
+F 0 "#PWR021" H 7550 4300 50  0001 C CNN
 F 1 "GND" H 7550 4400 50  0000 C CNN
 F 2 "" H 7550 4550 50  0001 C CNN
@@
 	8300 3550 8300 4050
 $Comp
-L +3V3 #PWR18
+L +3V3 #PWR022
 U 1 1 5AC2E6F2
 P 8300 3550
-F 0 "#PWR18" H 8300 3400 50  0001 C CNN
+F 0 "#PWR022" H 8300 3400 50  0001 C CNN
 F 1 "+3V3" H 8300 3690 50  0000 C CNN
 F 2 "" H 8300 3550 50  0001 C CNN
@@
 $EndComp
 $Comp
-L +5V #PWR15
+L +5V #PWR023
 U 1 1 5AC2E744
 P 6850 3550
-F 0 "#PWR15" H 6850 3400 50  0001 C CNN
+F 0 "#PWR023" H 6850 3400 50  0001 C CNN
 F 1 "+5V" H 6850 3690 50  0000 C CNN
 F 2 "" H 6850 3550 50  0001 C CNN
@@
 F 0 "PSU1" H 3300 1900 60  0000 L CNN
 F 1 "IRM-15-5" H 3300 1800 60  0000 L CNN
-F 2 "" H 3100 1650 60  0001 C CNN
+F 2 "opqbox3:IRM-15-5" H 3100 1650 60  0001 C CNN
 F 3 "" H 3100 1650 60  0001 C CNN
 	1    3100 1650

Commit message: Fix U1 for real this time
Parts:
- U1: footprint SMD_Packages:SOIC-8-N -> opqbox3:AMC1100DWV
Changed lines of the file:
@@
 F 0 "U1" H 3250 4050 60  0000 L CNN
 F 1 "AMC1100DWV" H 3250 3950 60  0000 L CNN
-F 2 "SMD_Packages:SOIC-8-N" H 3050 3800 60  0001 C CNN
+F 2 "opqbox3:AMC1100DWV" H 3050 3800 60  0001 C CNN
 F 3 "" H 3050 3800 60  0001 C CNN
 	1    3050 3800

Commit message: Moved brokers to rust with mongo reporting
Parts:
- C1, C10, C11, C12, C13, C2, C3, C4, C5, C6, C7, C8, C9: symbol C -> opqbox3-rescue:C
- F1, F2: symbol Fuse -> opqbox3-rescue:Fuse
- L1: symbol L -> opqbox3-rescue:L
- PSU1: symbol IRM-15-5 -> opqbox3-rescue:IRM-15-5
- PSU2: symbol ADUM5010ARSZ -> opqbox3-rescue:ADUM5010ARSZ
- R1, R2, R3, R4, R5, R6, R7, R8, R9: symbol R -> opqbox3-rescue:R
- REG1: symbol AP2120N-3.3TRG1 -> opqbox3-rescue:AP2120N-3.3TRG1
- RV1: symbol Varistor -> opqbox3-rescue:Varistor
- U1: symbol AMC1100DWV -> opqbox3-rescue:AMC1100DWV
- U3: symbol ISL21010CFH333Z-TK -> opqbox3-rescue:ISL21010CFH333Z-TK
Connections:
- wire segments 110 -> 162
